File: ergogen/kicad/skoldpad.kicad_pcb (KiCad board)
At the start: 2 copper layers, 141.9 x 109.3 mm, 94 parts

Commit message: Rename Signature.pretty footprint library to Skoldpad.pretty
More project-specific name for the custom footprint library, updated
in fp-lib-table, the routed PCB, CLAUDE.md, and README.

Co-Authored-By: Claude Sonnet 5 <noreply@anthropic.com>
Parts:
- G*** (x2): footprint Signature:shieldpad -> Skoldpad:shieldpad
- G*** (x2): footprint Signature:tank -> Skoldpad:tank
Changed lines of the file:
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@@
       (net 10 "main_index_bottom") (zone_connect 2))
   )
-  (footprint "Signature:shieldpad" (layer "F.Cu")
+  (footprint "Skoldpad:shieldpad" (layer "F.Cu")
     (at 124 120.7)
     (attr board_only exclude_from_pos_files exclude_from_bom)
@@
       (net 3 "main_outer_home"))
   )
-  (footprint "Signature:tank" (layer "F.Cu")
+  (footprint "Skoldpad:tank" (layer "F.Cu")
     (at 206.958546 110.670053)
     (attr board_only exclude_from_pos_files exclude_from_bom)
@@
       (net 13 "main_inner_bottom") (zone_connect 2))
   )
-  (footprint "Signature:shieldpad" (layer "B.Cu")
+  (footprint "Skoldpad:shieldpad" (layer "B.Cu")
     (at 124 120.7 180)
     (attr board_only exclude_from_pos_files exclude_from_bom)
@@
       (stroke (width 0) (type solid)) (fill solid) (layer "B.Mask"))
   )
-  (footprint "Signature:tank" (layer "B.Cu")
+  (footprint "Skoldpad:tank" (layer "B.Cu")
     (at 206.958546 110.670053 180)
     (attr board_only exclude_from_pos_files exclude_from_bom)
